Commit message: Update dami2.urdf.xacro

File: dami2_description/urdf/dami2.urdf.xacro (robot description, xacro)
@@ -163,5 +163,5 @@
     <origin xyz="-0.054025 0.0 0.14405" rpy="0 0 0"/>
   </joint>
-  <link name="base_scan">
+  <link name="camera_link">
     <inertial>
       <mass value="0.114" />
@@ -185,5 +185,5 @@
     </collision>
   </link>
-<!--  <joint name="camera_depth_joint" type="fixed">
+  <joint name="camera_depth_joint" type="fixed">
     <origin xyz="0 0.01235 0.0" rpy="0 0 0" />
     <parent link="camera_link" />
@@ -209,4 +209,3 @@
   </joint>
   <link name="camera_rgb_optical_frame"/>
--->
 </robot>

Commit message: Update dami2.urdf.xacro

File: dami2_description/urdf/dami2.urdf.xacro (robot description, xacro)
@@ -171,5 +171,5 @@
                izz="0.001" />
     </inertial>
-<!--    <visual>
+    <visual>
       <origin xyz="0 0 0 " rpy="0 0 1.570796" />
       <geometry>
@@ -177,5 +177,5 @@
       </geometry>
       <material name="dark"/>
-    </visual>-->
+    </visual>
     <collision>
       <origin xyz="0 0 0" rpy="0 0 0" />

Commit message: Update dami2.urdf.xacro

File: dami2_description/urdf/dami2.urdf.xacro (robot description, xacro)
@@ -160,5 +160,5 @@
   <joint name="scan_joint" type="fixed">
     <parent link="base_link"/>
-    <child link="base_scan"/>
+    <child link="camera_link"/>
     <origin xyz="-0.054025 0.0 0.14405" rpy="0 0 0"/>
   </joint>
